File: kicad/four_pack/four_cells.kicad_pcb (KiCad board)
At the start: 2 copper layers, 80 x 81 mm, 35 parts, among them J1 cell_+, J10 bal_even_right, J11 bal_odd_right, J12 cell_+, J13 cell_+, J14 bal_odd_right, J15 bal_even_right, J2 cell_-, J3 bal_even_left, J4 bal_even_right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

Commit message: Small change
Parts:
- moved H1 1.00 mm to (14.5, 16.0)
- moved H10 1.00 mm to (69.5, 16.0)
- moved H11 1.00 mm to (54.5, 89.0)
- moved H12 1.00 mm to (69.5, 89.0)
- moved H13 1.00 mm to (74.5, 16.0)
- moved H14 1.00 mm to (89.5, 16.0)
- moved H15 1.00 mm to (74.5, 89.0)
- moved H16 1.00 mm to (89.5, 89.0)
- moved H2 1.00 mm to (29.5, 16.0)
- moved H3 1.00 mm to (29.5, 89.0)
- moved H4 1.00 mm to (14.5, 89.0)
- moved H6 1.00 mm to (49.5, 16.0)
- moved H7 1.00 mm to (34.5, 89.0)
- moved H8 1.00 mm to (49.5, 89.0)
- moved H9 1.00 mm to (54.5, 16.0)
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Other:
- board size 80 x 81 mm -> 80 x 75 mm

Commit message: Ending PCB finished
Parts:
- added J16: communication, telec:DualSide_2x05_P1.27mm_Vertical_SMD, F.Cu at (12.0, 52.6)
- added J17: communication, telec:DualSide_2x05_P1.27mm_Vertical_SMD, F.Cu at (32.0, 52.6)
- added J18: communication, telec:DualSide_2x05_P1.27mm_Vertical_SMD, F.Cu at (52.0, 52.6)
- added J19: communication, telec:DualSide_2x05_P1.27mm_Vertical_SMD, F.Cu at (72.0, 52.6)
- added J20: communication, telec:DualSide_2x05_P1.27mm_Vertical_SMD, F.Cu at (92.0, 52.6)
Routing:
- net Net-(J16-Pad8): track 0.00 -> 80.0 mm
- net Net-(J16-Pad7): track 0.00 -> 80.0 mm
- net Net-(J16-Pad6): track 0.00 -> 80.0 mm
- net Net-(J16-Pad5): track 0.00 -> 80.0 mm
- net Net-(J16-Pad4): track 0.00 -> 80.0 mm
- net Net-(J16-Pad3): track 0.00 -> 80.0 mm
- net Net-(J16-Pad2): track 0.00 -> 80.0 mm
- net Net-(J16-Pad1): track 0.00 -> 80.0 mm
