File: kicad/four_pack/four_cells.kicad_pcb (KiCad board)
At the start: 2 copper layers, 80 x 75 mm, 44 parts, among them J1 cell_+, J10 bal_even_right, J11 bal_odd_right, J12 cell_+, J13 cell_+, J14 bal_odd_right, J15 bal_even_right, J16 communication, J17 communication, J18 communication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

Commit message: Updated to kicad 7.x
Connections:
- J3 pad 8: Net-(J3-Pad8) -> unconnected-(J3-Pin_8-Pad8)
Other:
- net class Default removed
