File: kicad/four_pack/four_cells.sch (KiCad schematic (older format))
At the start: 40 parts, among them J1 cell_+, J10 bal_even_right, J11 bal_odd_right, J12 cell_+, J13 cell_+, J14 bal_odd_right, J15 bal_even_right, J16 communication, J17 communication, J18 communication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

Commit message: gerber + logo
Parts:
- added LOGO1, LOGO? (x3): Logo_Open_Hardware_Small, logo:batpacked-24, symbol Graphic:Logo_Open_Hardware_Small
Changed lines of the file:
@@
 Wire Wire Line
 	7750 4050 10450 4050
+$Comp
+L Graphic:Logo_Open_Hardware_Small LOGO1
+U 1 1 60FFB8ED
+P 7350 6800
+F 0 "LOGO1" H 7350 7075 50  0001 C CNN
+F 1 "Logo_Open_Hardware_Small" H 7350 6575 50  0001 C CNN
+F 2 "logo:batpacked-24" H 7350 6800 50  0001 C CNN
+F 3 "~" H 7350 6800 50  0001 C CNN
+	1    7350 6800
+	1    0    0    -1
+$EndComp
+$Comp
+L Graphic:Logo_Open_Hardware_Small LOGO?
+U 1 1 610045D6
+P 7850 6850
+F 0 "LOGO?" H 7850 7125 50  0001 C CNN
+F 1 "Logo_Open_Hardware_Small" H 7850 6625 50  0001 C CNN
+F 2 "logo:batpacked-24" H 7850 6850 50  0001 C CNN
+F 3 "~" H 7850 6850 50  0001 C CNN
+	1    7850 6850
+	1    0    0    -1
+$EndComp
+$Comp
+L Graphic:Logo_Open_Hardware_Small LOGO?
+U 1 1 61004A09
+P 8400 6850
+F 0 "LOGO?" H 8400 7125 50  0001 C CNN
+F 1 "Logo_Open_Hardware_Small" H 8400 6625 50  0001 C CNN
+F 2 "logo:batpacked-24" H 8400 6850 50  0001 C CNN
+F 3 "~" H 8400 6850 50  0001 C CNN
+	1    8400 6850
+	1    0    0    -1
+$EndComp
+$Comp
+L Graphic:Logo_Open_Hardware_Small LOGO?
+U 1 1 61004EF1
+P 9200 6900
+F 0 "LOGO?" H 9200 7175 50  0001 C CNN
+F 1 "Logo_Open_Hardware_Small" H 9200 6675 50  0001 C CNN
+F 2 "logo:batpacked-24" H 9200 6900 50  0001 C CNN
+F 3 "~" H 9200 6900 50  0001 C CNN
+	1    9200 6900
+	1    0    0    -1
+$EndComp
 $EndSCHEMATC

Commit message: gerber + logo
Parts:
- gave numbers to parts that had none: 3
Changed lines of the file:
@@
 $EndComp
 $Comp
-L Graphic:Logo_Open_Hardware_Small LOGO?
+L Graphic:Logo_Open_Hardware_Small LOGO2
 U 1 1 610045D6
 P 7850 6850
-F 0 "LOGO?" H 7850 7125 50  0001 C CNN
+F 0 "LOGO2" H 7850 7125 50  0001 C CNN
 F 1 "Logo_Open_Hardware_Small" H 7850 6625 50  0001 C CNN
 F 2 "logo:batpacked-24" H 7850 6850 50  0001 C CNN
@@
 $EndComp
 $Comp
-L Graphic:Logo_Open_Hardware_Small LOGO?
+L Graphic:Logo_Open_Hardware_Small LOGO3
 U 1 1 61004A09
 P 8400 6850
-F 0 "LOGO?" H 8400 7125 50  0001 C CNN
+F 0 "LOGO3" H 8400 7125 50  0001 C CNN
 F 1 "Logo_Open_Hardware_Small" H 8400 6625 50  0001 C CNN
 F 2 "logo:batpacked-24" H 8400 6850 50  0001 C CNN
@@
 $EndComp
 $Comp
-L Graphic:Logo_Open_Hardware_Small LOGO?
+L Graphic:Logo_Open_Hardware_Small LOGO4
 U 1 1 61004EF1
 P 9200 6900
-F 0 "LOGO?" H 9200 7175 50  0001 C CNN
+F 0 "LOGO4" H 9200 7175 50  0001 C CNN
 F 1 "Logo_Open_Hardware_Small" H 9200 6675 50  0001 C CNN
 F 2 "logo:batpacked-24" H 9200 6900 50  0001 C CNN
