File: kicad/BMS/BMS.sch (KiCad schematic (older format))
At the start: 23 parts, among them J1 cells_+, J16 communication, J2 cells_-, J3 bal_even_left, J5 bal_odd_left

Commit message: More on the charger
Parts:
- added L?: 1u, symbol Device:L
- D?: value D_Schottky -> MBR0520
- J3: value bal_even_left -> bal_even
- J5: value bal_odd_left -> bal_odd
- R?: value R -> 2M2
- R?: value R -> 100k
- R?: value 13k -> 0
Connections:
- wire segments 25 -> 31
Other:
- moved on the sheet: J3, J5, R?, U?
Changed lines of the file:
@@
 L Connector:Conn_01x08_Male J5
 U 1 1 608882E0
-P 8350 3500
-F 0 "J5" H 8450 4000 50  0000 C CNN
-F 1 "bal_odd_left" H 8458 3890 50  0000 C CNN
-F 2 "telec:Castellated_1x08_P2.54mm" H 8350 3500 50  0001 C CNN
-F 3 "~" H 8350 3500 50  0001 C CNN
-	1    8350 3500
+P 9300 3550
+F 0 "J5" H 9400 4050 50  0000 C CNN
+F 1 "bal_odd" H 9408 3940 50  0000 C CNN
+F 2 "telec:Castellated_1x08_P2.54mm" H 9300 3550 50  0001 C CNN
+F 3 "~" H 9300 3550 50  0001 C CNN
+	1    9300 3550
 	-1   0    0    -1
 $EndComp
@@
 L Connector:Conn_01x08_Male J3
 U 1 1 6088705C
-P 8350 2450
-F 0 "J3" H 8500 2950 50  0000 R CNN
-F 1 "bal_even_left" H 8650 2850 50  0000 R CNN
-F 2 "telec:Castellated_1x08_P2.54mm" H 8350 2450 50  0001 C CNN
-F 3 "~" H 8350 2450 50  0001 C CNN
-	1    8350 2450
-	-1   0    0    -1
+P 9300 2500
+F 0 "J3" H 9450 3000 50  0000 R CNN
+F 1 "bal_even" H 9600 2900 50  0000 R CNN
+F 2 "telec:Castellated_1x08_P2.54mm" H 9300 2500 50  0001 C CNN
+F 3 "~" H 9300 2500 50  0001 C CNN
+	1    9300 2500
+	-1   0    0    1
 $EndComp
 $Comp
@@
 L telec:BQ76942 U?
 U 1 1 60AD0042
-P 6750 2950
-F 0 "U?" H 7300 4450 50  0000 C CNN
-F 1 "BQ76942" H 6200 4450 50  0000 C CNN
-F 2 "Package_QFP:TQFP-48_7x7mm_P0.5mm" V 6800 2950 50  0001 C CNN
-F 3 "http://www.ti.com/lit/gpn/bq76940" H 7450 4100 50  0001 C CNN
-	1    6750 2950
+P 6750 2850
+F 0 "U?" H 7300 4350 50  0000 C CNN
+F 1 "BQ76942" H 6200 4350 50  0000 C CNN
+F 2 "Package_QFP:TQFP-48_7x7mm_P0.5mm" V 6800 2850 50  0001 C CNN
+F 3 "http://www.ti.com/lit/gpn/bq76940" H 7450 4000 50  0001 C CNN
+	1    6750 2850
 	1    0    0    -1
 $EndComp
@@
 P 3200 2200
 F 0 "D?" H 3200 1984 50  0000 C CNN
-F 1 "D_Schottky" H 3200 2075 50  0000 C CNN
+F 1 "MBR0520" H 3200 2075 50  0000 C CNN
 F 2 "" H 3200 2200 50  0001 C CNN
 F 3 "~" H 3200 2200 50  0001 C CNN
@@
 P 3950 2800
 F 0 "R?" H 4020 2846 50  0000 L CNN
-F 1 "R" H 4020 2755 50  0000 L CNN
+F 1 "2M2" H 4020 2755 50  0000 L CNN
 F 2 "" V 3880 2800 50  0001 C CNN
 F 3 "~" H 3950 2800 50  0001 C CNN
@@
 P 3950 3300
 F 0 "R?" H 4020 3346 50  0000 L CNN
-F 1 "R" H 4020 3255 50  0000 L CNN
+F 1 "100k" H 4020 3255 50  0000 L CNN
 F 2 "" V 3880 3300 50  0001 C CNN
 F 3 "~" H 3950 3300 50  0001 C CNN
@@
 L Device:R_Small R?
 U 1 1 60AFF798
-P 2150 3250
-F 0 "R?" H 2300 3300 50  0000 R CNN
-F 1 "13k" H 2350 3200 50  0000 R CNN
-F 2 "" H 2150 3250 50  0001 C CNN
-F 3 "~" H 2150 3250 50  0001 C CNN
-	1    2150 3250
+P 2250 3250
+F 0 "R?" H 2400 3300 50  0000 R CNN
+F 1 "0" H 2400 3200 50  0000 R CNN
+F 2 "" H 2250 3250 50  0001 C CNN
+F 3 "~" H 2250 3250 50  0001 C CNN
+	1    2250 3250
 	-1   0    0    -1
 $EndComp
@@
 L power:GND #PWR?
 U 1 1 60B05FF4
-P 2150 3550
-F 0 "#PWR?" H 2150 3300 50  0001 C CNN
-F 1 "GND" H 2155 3377 50  0000 C CNN
-F 2 "" H 2150 3550 50  0001 C CNN
-F 3 "" H 2150 3550 50  0001 C CNN
-	1    2150 3550
-	1    0    0    -1
-$EndComp
-Wire Wire Line
-	2150 3550 2150 3350
+P 2250 3550
+F 0 "#PWR?" H 2250 3300 50  0001 C CNN
+F 1 "GND" H 2255 3377 50  0000 C CNN
+F 2 "" H 2250 3550 50  0001 C CNN
+F 3 "" H 2250 3550 50  0001 C CNN
+	1    2250 3550
+	1    0    0    -1
+$EndComp
+Wire Wire Line
+	2250 3550 2250 3350
 Wire Wire Line
 	2800 3550 2800 3450
@@
 $EndComp
 Wire Wire Line
-	2150 3150 2150 2900
-Wire Wire Line
-	2150 2900 2300 2900
+	2250 3150 2250 2900
+Wire Wire Line
+	2250 2900 2300 2900
 Wire Wire Line
 	2300 2800 2250 2800
@@
 Wire Wire Line
 	3400 2200 3350 2200
+Wire Wire Line
+	9100 2800 8450 2800
+Wire Wire Line
+	8450 2800 8450 3650
+Wire Wire Line
+	8450 3650 7550 3650
+$Comp
+L Device:L L?
+U 1 1 60B78898
+P 4300 2200
+F 0 "L?" V 4490 2200 50  0000 C CNN
+F 1 "1u" V 4399 2200 50  0000 C CNN
+F 2 "" H 4300 2200 50  0001 C CNN
+F 3 "~" H 4300 2200 50  0001 C CNN
+	1    4300 2200
+	0    -1   -1   0
+$EndComp
+Wire Wire Line
+	3950 2200 4150 2200
+Wire Wire Line
+	4450 2200 4650 2200
+Connection ~ 3950 2200
+Wire Wire Line
+	2250 2200 1950 2200
+Connection ~ 2250 2200
 $EndSCHEMATC
