File: kicad/end_pack/end_pack.sch (KiCad schematic (older format))
At the start: 40 parts, among them J1 cell_+, J10 bal_even_right, J11 bal_odd_right, J12 cell_+, J13 cell_+, J14 bal_odd_right, J15 bal_even_right, J16 communication, J17 communication, J18 communication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

Commit message: Ending PCB finished
Parts:
- removed BT1: Battery_Cell, telec:Cell_18650, symbol Device:Battery_Cell
- removed H1, H3: MountingHole, MountingHole:MountingHole_2mm, symbol Mechanical:MountingHole
- removed J16: communication, telec:DualSide_2x05_P1.27mm_Vertical_SMD, symbol Connector:Conn_01x08_Male
- removed J2: cell_-, telec:Castellated_1x01_P5.08mm_Double, symbol Connector:Conn_01x01_Male
- removed J3: bal_even_left, telec:Castellated_1x08_P2.54mm, symbol Connector:Conn_01x08_Male
- removed J5: bal_odd_left, telec:Castellated_1x08_P2.54mm, symbol Connector:Conn_01x08_Male
- added D1, D2, D3, D4, D5, D6: LED, LED_SMD:LED_1206_3216Metric, symbol Device:LED
- added J2: cell_+, Connector_Pin:Pin_D1.3mm_L11.0mm_LooseFit, symbol Connector:Conn_01x01_Female
- added R1, R2, R3, R4, R5, R6: 1k, Resistor_SMD:R_0805_2012Metric, symbol Device:R
- added SW1: SW_Push, Button_Switch_SMD:SW_Push_SPST_NO_Alps_SKRK, symbol Switch:SW_Push
Connections:
- net labels added: GND
- wire segments 176 -> 157
- no-connect marks 1 -> 0

Commit message: gerber + logo
Parts:
- added LOGO1, LOGO2, LOGO3: Logo_Open_Hardware_Small, logo:batpacked-24, symbol Graphic:Logo_Open_Hardware_Small
Changed lines of the file:
@@
 Connection ~ 2250 4650
 Connection ~ 2250 4750
+$Comp
+L Graphic:Logo_Open_Hardware_Small LOGO1
+U 1 1 60FFA3B6
+P 7300 6850
+F 0 "LOGO1" H 7300 7125 50  0001 C CNN
+F 1 "Logo_Open_Hardware_Small" H 7300 6625 50  0001 C CNN
+F 2 "logo:batpacked-24" H 7300 6850 50  0001 C CNN
+F 3 "~" H 7300 6850 50  0001 C CNN
+	1    7300 6850
+	1    0    0    -1
+$EndComp
+$Comp
+L Graphic:Logo_Open_Hardware_Small LOGO3
+U 1 1 60FFBE01
+P 7850 6800
+F 0 "LOGO3" H 7850 7075 50  0001 C CNN
+F 1 "Logo_Open_Hardware_Small" H 7850 6575 50  0001 C CNN
+F 2 "logo:batpacked-24" H 7850 6800 50  0001 C CNN
+F 3 "~" H 7850 6800 50  0001 C CNN
+	1    7850 6800
+	1    0    0    -1
+$EndComp
+$Comp
+L Graphic:Logo_Open_Hardware_Small LOGO2
+U 1 1 60FFC411
+P 8550 6700
+F 0 "LOGO2" H 8550 6975 50  0001 C CNN
+F 1 "Logo_Open_Hardware_Small" H 8550 6475 50  0001 C CNN
+F 2 "logo:batpacked-24" H 8550 6700 50  0001 C CNN
+F 3 "~" H 8550 6700 50  0001 C CNN
+	1    8550 6700
+	1    0    0    -1
+$EndComp
 $EndSCHEMATC
