File: kicad/end_pack/end_pack.kicad_pcb (KiCad board)
At the start: 2 copper layers, 70 x 75 mm, 50 parts, among them J1 cell_+, J10 bal_even_right, J11 bal_odd_right, J12 cell_+, J13 cell_+, J14 bal_odd_right, J15 bal_even_right, J17 communication, J18 communication, J19 communication, J2 cell_+, J20 communication, J4 bal_even_right, J6 bal_odd_right, J7 cell_+, J8 bal_odd_right, J9 bal_even_right, SW1 SW_Push

Commit message: Updated to kicad 7.x
Connections:
- BT2 pad 1: Net-(BT2-Pad1) -> Net-(BT2-+)
- BT2 pad 2: Net-(BT2-Pad2) -> Net-(BT2--)
- BT3 pad 1: Net-(BT3-Pad1) -> Net-(BT3-+)
- BT3 pad 2: Net-(BT2-Pad1) -> Net-(BT2-+)
- BT4 pad 2: Net-(BT3-Pad1) -> Net-(BT3-+)
- J1 pad 1: Net-(BT2-Pad2) -> unconnected-(J1-Pin_1-Pad1)
- J10 pad 1: Net-(BT3-Pad1) -> unconnected-(J10-Pin_1-Pad1)
- J10 pad 2: Net-(BT2-Pad2) -> unconnected-(J10-Pin_2-Pad2)
- J10 pad 3: Net-(J10-Pad3) -> unconnected-(J10-Pin_3-Pad3)
- J10 pad 4: Net-(J10-Pad4) -> unconnected-(J10-Pin_4-Pad4)
- J10 pad 5: Net-(J10-Pad5) -> unconnected-(J10-Pin_5-Pad5)
- J10 pad 6: Net-(J10-Pad6) -> unconnected-(J10-Pin_6-Pad6)
- J10 pad 7: Net-(J10-Pad7) -> unconnected-(J10-Pin_7-Pad7)
- J10 pad 8: Net-(J10-Pad8) -> unconnected-(J10-Pin_8-Pad8)
- J11 pad 1: Net-(BT2-Pad1) -> unconnected-(J11-Pin_1-Pad1)
- J11 pad 2: Net-(J11-Pad2) -> unconnected-(J11-Pin_2-Pad2)
- J11 pad 3: Net-(J11-Pad3) -> unconnected-(J11-Pin_3-Pad3)
- J11 pad 4: Net-(J11-Pad4) -> unconnected-(J11-Pin_4-Pad4)
- J11 pad 5: Net-(J11-Pad5) -> unconnected-(J11-Pin_5-Pad5)
- J11 pad 6: Net-(J11-Pad6) -> unconnected-(J11-Pin_6-Pad6)
- J11 pad 7: Net-(J11-Pad7) -> unconnected-(J11-Pin_7-Pad7)
- J11 pad 8: Net-(J11-Pad8) -> Net-(J11-Pin_8)
- J12 pad 1: Net-(BT3-Pad1) -> unconnected-(J12-Pin_1-Pad1)
- J14 pad 1: Net-(BT3-Pad1) -> Net-(BT3-+)
- J14 pad 2: Net-(BT2-Pad2) -> Net-(BT2--)
- J14 pad 3: Net-(J10-Pad3) -> Net-(J14-Pin_3)
- J14 pad 4: Net-(J10-Pad4) -> Net-(J14-Pin_4)
- J14 pad 5: Net-(J10-Pad5) -> Net-(J14-Pin_5)
- J14 pad 6: Net-(J10-Pad6) -> Net-(J14-Pin_6)
- J14 pad 7: Net-(J10-Pad7) -> Net-(J14-Pin_7)
- J14 pad 8: Net-(J10-Pad8) -> Net-(J14-Pin_8)
- J15 pad 2: Net-(BT2-Pad1) -> Net-(BT2-+)
- J15 pad 3: Net-(J11-Pad2) -> Net-(J15-Pin_3)
- J15 pad 4: Net-(J11-Pad3) -> Net-(J15-Pin_4)
- J15 pad 5: Net-(J11-Pad4) -> Net-(J15-Pin_5)
- J15 pad 6: Net-(J11-Pad5) -> Net-(J15-Pin_6)
- J15 pad 7: Net-(J11-Pad6) -> Net-(J15-Pin_7)
- J15 pad 8: Net-(J11-Pad7) -> Net-(J15-Pin_8)
- J17 pad 1: Net-(J17-Pad1) -> unconnected-(J17-Pin_1-Pad1)
- J17 pad 2: Net-(J17-Pad2) -> unconnected-(J17-Pin_2-Pad2)
- J17 pad 3: Net-(J17-Pad3) -> unconnected-(J17-Pin_3-Pad3)
- J17 pad 4: Net-(J17-Pad4) -> unconnected-(J17-Pin_4-Pad4)
- J17 pad 5: GND -> unconnected-(J17-Pin_5-Pad5)
- J17 pad 6: Net-(J17-Pad6) -> unconnected-(J17-Pin_6-Pad6)
- J17 pad 7: Net-(J17-Pad7) -> unconnected-(J17-Pin_7-Pad7)
- J17 pad 8: Net-(J17-Pad8) -> unconnected-(J17-Pin_8-Pad8)
- J18 pad 1: Net-(J17-Pad1) -> unconnected-(J18-Pin_1-Pad1)
- J18 pad 2: Net-(J17-Pad2) -> unconnected-(J18-Pin_2-Pad2)
- J18 pad 3: Net-(J17-Pad3) -> unconnected-(J18-Pin_3-Pad3)
- J18 pad 4: Net-(J17-Pad4) -> unconnected-(J18-Pin_4-Pad4)
- J18 pad 5: GND -> unconnected-(J18-Pin_5-Pad5)
- J18 pad 6: Net-(J17-Pad6) -> unconnected-(J18-Pin_6-Pad6)
- J18 pad 7: Net-(J17-Pad7) -> unconnected-(J18-Pin_7-Pad7)
- J18 pad 8: Net-(J17-Pad8) -> unconnected-(J18-Pin_8-Pad8)
- J19 pad 1: Net-(J17-Pad1) -> unconnected-(J19-Pin_1-Pad1)
- J19 pad 2: Net-(J17-Pad2) -> unconnected-(J19-Pin_2-Pad2)
- J19 pad 3: Net-(J17-Pad3) -> unconnected-(J19-Pin_3-Pad3)
- J19 pad 4: Net-(J17-Pad4) -> unconnected-(J19-Pin_4-Pad4)
- J19 pad 5: GND -> unconnected-(J19-Pin_5-Pad5)
- J19 pad 6: Net-(J17-Pad6) -> unconnected-(J19-Pin_6-Pad6)
- J19 pad 7: Net-(J17-Pad7) -> unconnected-(J19-Pin_7-Pad7)
- J19 pad 8: Net-(J17-Pad8) -> unconnected-(J19-Pin_8-Pad8)
- J2 pad 1: Net-(BT2-Pad2) -> Net-(BT2--)
- J20 pad 1: Net-(J17-Pad1) -> Net-(J20-Pin_1)
- J20 pad 2: Net-(J17-Pad2) -> Net-(J20-Pin_2)
- J20 pad 3: Net-(J17-Pad3) -> Net-(J20-Pin_3)
- J20 pad 4: Net-(J17-Pad4) -> Net-(J20-Pin_4)
- J20 pad 6: Net-(J17-Pad6) -> Net-(J20-Pin_6)
- J20 pad 7: Net-(J17-Pad7) -> Net-(J20-Pin_7)
- J20 pad 8: Net-(J17-Pad8) -> Net-(J20-Pin_8)
- J4 pad 1: Net-(BT2-Pad2) -> unconnected-(J4-Pin_1-Pad1)
- J4 pad 2: Net-(J10-Pad3) -> Net-(J14-Pin_3)
- J4 pad 3: Net-(J10-Pad4) -> Net-(J14-Pin_4)
- J4 pad 4: Net-(J10-Pad5) -> Net-(J14-Pin_5)
- J4 pad 5: Net-(J10-Pad6) -> Net-(J14-Pin_6)
- J4 pad 6: Net-(J10-Pad7) -> Net-(J14-Pin_7)
- J4 pad 7: Net-(J10-Pad8) -> Net-(J14-Pin_8)
- J6 pad 1: Net-(J11-Pad2) -> Net-(J15-Pin_3)
- J6 pad 2: Net-(J11-Pad3) -> Net-(J15-Pin_4)
- J6 pad 3: Net-(J11-Pad4) -> Net-(J15-Pin_5)
- J6 pad 4: Net-(J11-Pad5) -> Net-(J15-Pin_6)
- J6 pad 5: Net-(J11-Pad6) -> Net-(J15-Pin_7)
- J6 pad 6: Net-(J11-Pad7) -> Net-(J15-Pin_8)
- J6 pad 7: Net-(J11-Pad8) -> Net-(J11-Pin_8)
- J6 pad 8: Net-(J6-Pad8) -> unconnected-(J6-Pin_8-Pad8)
- J7 pad 1: Net-(BT2-Pad1) -> unconnected-(J7-Pin_1-Pad1)
- J8 pad 1: Net-(BT2-Pad2) -> unconnected-(J8-Pin_1-Pad1)
- J8 pad 2: Net-(J10-Pad3) -> unconnected-(J8-Pin_2-Pad2)
- J8 pad 3: Net-(J10-Pad4) -> unconnected-(J8-Pin_3-Pad3)
- J8 pad 4: Net-(J10-Pad5) -> unconnected-(J8-Pin_4-Pad4)
- J8 pad 5: Net-(J10-Pad6) -> unconnected-(J8-Pin_5-Pad5)
- J8 pad 6: Net-(J10-Pad7) -> unconnected-(J8-Pin_6-Pad6)
- J8 pad 7: Net-(J10-Pad8) -> unconnected-(J8-Pin_7-Pad7)
- J9 pad 1: Net-(BT2-Pad1) -> unconnected-(J9-Pin_1-Pad1)
- J9 pad 2: Net-(J11-Pad2) -> unconnected-(J9-Pin_2-Pad2)
- J9 pad 3: Net-(J11-Pad3) -> unconnected-(J9-Pin_3-Pad3)
- J9 pad 4: Net-(J11-Pad4) -> unconnected-(J9-Pin_4-Pad4)
- J9 pad 5: Net-(J11-Pad5) -> unconnected-(J9-Pin_5-Pad5)
- J9 pad 6: Net-(J11-Pad6) -> unconnected-(J9-Pin_6-Pad6)
- J9 pad 7: Net-(J11-Pad7) -> unconnected-(J9-Pin_7-Pad7)
- J9 pad 8: Net-(J11-Pad8) -> unconnected-(J9-Pin_8-Pad8)
- R1 pad 2: Net-(J17-Pad1) -> Net-(J20-Pin_1)
- R2 pad 2: Net-(J17-Pad4) -> Net-(J20-Pin_4)
- R3 pad 2: Net-(J17-Pad3) -> Net-(J20-Pin_3)
- R4 pad 2: Net-(J17-Pad6) -> Net-(J20-Pin_6)
- R5 pad 2: Net-(J17-Pad7) -> Net-(J20-Pin_7)
- R6 pad 2: Net-(J17-Pad8) -> Net-(J20-Pin_8)
- SW1 pad 1: Net-(J17-Pad2) -> Net-(J20-Pin_2)
Routing:
- net Net-(J20-Pin_2): track 0.00 -> 74.1 mm, vias 0 -> 1
- net Net-(J17-Pad2): track 74.1 -> 0.00 mm, vias 1 -> 0
- net Net-(BT2-Pad2): track 73.9 -> 0.00 mm
- net Net-(BT2--): track 0.00 -> 73.9 mm
- net Net-(J20-Pin_8): track 0.00 -> 66.0 mm, vias 0 -> 1
- net Net-(J17-Pad8): track 66.0 -> 0.00 mm, vias 1 -> 0
- net Net-(J20-Pin_1): track 0.00 -> 65.2 mm
- net Net-(J17-Pad1): track 65.2 -> 0.00 mm
- net Net-(J20-Pin_4): track 0.00 -> 65.2 mm, vias 0 -> 1
- net Net-(J17-Pad4): track 65.2 -> 0.00 mm, vias 1 -> 0
- net Net-(J20-Pin_7): track 0.00 -> 63.2 mm
- net Net-(J17-Pad7): track 63.2 -> 0.00 mm
- net Net-(J20-Pin_3): track 0.00 -> 62.9 mm
- net Net-(J17-Pad3): track 62.9 -> 0.00 mm
- net Net-(J20-Pin_6): track 0.00 -> 62.8 mm, vias 0 -> 1
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- added copper zone on B.Cu, net Net-(BT2-+)
- added copper zone on F.Cu, net Net-(BT2-+)
- added copper zone on B.Cu, net Net-(BT2--)
- added copper zone on F.Cu, net Net-(BT2--)
- added copper zone on B.Cu, net Net-(BT3-+)
- added copper zone on F.Cu, net Net-(BT3-+)
- removed copper zone on B.Cu, net Net-(BT2-Pad1)
- removed copper zone on F.Cu, net Net-(BT2-Pad1)
- removed copper zone on B.Cu, net Net-(BT2-Pad2)
- removed copper zone on F.Cu, net Net-(BT2-Pad2)
- removed copper zone on B.Cu, net Net-(BT3-Pad1)
- removed copper zone on F.Cu, net Net-(BT3-Pad1)
Other:
- board size 70 x 75 mm -> 71.9 x 75 mm
- net class Default removed
