File: kicad/single_cell/stackable_cells_self_contained.sch (KiCad schematic (older format))
At the start: 20 parts, among them J1 cell_+, J2 cell_-, J3 bal_even_left, J4 bal_even_right, J5 bal_odd_left, J6 bal_odd_right, Q1 Q_NMOS_DGS, Q2 Q_NMOS_DGS, Q3 Q_NMOS_DGS, U1 FS312F-G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

Commit message: finished stackable design
Parts:
- added J16: communication, telec:DualSide_2x05_P1.27mm_Vertical_SMD, symbol Connector:Conn_01x08_Male
- added J17: communication, telec:DualSide_2x05_P1.27mm_Vertical_SMD, symbol Connector:Conn_01x08_Female
- J1: footprint Connector_PinSocket_2.54mm:PinSocket_1x01_P2.54mm_Horizontal -> telec:Castellated_1x01_P5.08mm_Double
- J2: footprint Connector_PinHeader_2.54mm:PinHeader_1x01_P2.54mm_Horizontal -> telec:Castellated_1x01_P5.08mm_Double
- J3, J5: footprint Connector_PinHeader_2.54mm:PinHeader_1x08_P2.54mm_Horizontal -> telec:Castellated_1x08_P2.54mm
- J4, J6: footprint Connector_PinSocket_2.54mm:PinSocket_1x08_P2.54mm_Horizontal -> telec:Castellated_1x08_P2.54mm
- Q1, Q2: value Q_NMOS_DGS -> Q_NMOS_GDS; symbol Device:Q_NMOS_DGS -> Device:Q_NMOS_GDS
- Q3: value Q_NMOS_DGS -> Q_NMOS_GSD; symbol Device:Q_NMOS_DGS -> Device:Q_NMOS_GSD
Connections:
- wire segments 61 -> 69
Other:
- moved on the sheet: BT1, C1, H3, H4, R1, R2, R3, U1, U2
