File: kicad/single_cell/stackable_cells.kicad_pcb (KiCad board)
At the start: 2 copper layers, 20 x 81 mm, 11 parts, among them J1 cell_+, J2 cell_-, J3 bal_even_left, J4 bal_even_right, J5 bal_odd_left, J6 bal_odd_right

Commit message: Updated to kicad 7.x
Connections:
- J3 pad 8: Net-(J3-Pad8) -> unconnected-(J3-Pin_8-Pad8)
Other:
- net class Default removed
